Commit message: fix dimensions of bottom legs

File: cheetah/cheetah.urdf (robot description, URDF)
Before this commit: robot cheetah, 11 links, 10 joints
Links:
- link bl_hip: mass 0.39061 -> 0.40409
- link bl_knee: mass 0.10247 -> 0.191716257710722
- link br_hip: mass 0.39061 -> 0.404107705466589
- link br_knee: mass 0.10247 -> 0.191716257710722
Joints:
- joint bl_knee_joint: origin xyz=0 0 -0.2 rpy=0 -0.5236 0 -> xyz=0 0 -0.21 rpy=0 -0.5236 0
- joint br_knee_joint: origin xyz=0 0 -0.2 rpy=0 -0.5236 0 -> xyz=0 0 -0.21 rpy=0 -0.5236 0
